Commit message: Add resend program interfaces into ros2_control xacro.

File: ur_description/urdf/ur.ros2_control.xacro (robot description, xacro)
@@ -136,4 +136,8 @@
         <command_interface name="target_speed_fraction_cmd"/>
         <command_interface name="target_speed_fraction_async_success"/>
+      </joint>
+      <joint name="resend_robot_program">
+        <command_interface name="resend_robot_program_cmd"/>
+        <command_interface name="resend_robot_program_async_success"/>
       </joint>
       <joint name="gpio">

Commit message: Make headless mode work in ursim.

File: ur_description/urdf/ur.ros2_control.xacro (robot description, xacro)
@@ -137,8 +137,4 @@
         <command_interface name="target_speed_fraction_cmd"/>
         <command_interface name="target_speed_fraction_async_success"/>
-      </joint>
-      <joint name="resend_robot_program">
-        <command_interface name="resend_robot_program_cmd"/>
-        <command_interface name="resend_robot_program_async_success"/>
       </joint>
       <joint name="gpio">

File: ur_description/urdf/ur.urdf.xacro (robot description, xacro)
@@ -31,5 +31,5 @@
      safety_k_position="$(arg safety_k_position)"
      use_fake_hardware="$(arg use_fake_hardware)"
-     fake_sensor_commands="$(arg fake_sensor_commands)
+     fake_sensor_commands="$(arg fake_sensor_commands)"
      headless_mode="$(arg headless_mode)" />
 </robot>

Commit message: pulling latest changes

File: ur_description/urdf/ur.ros2_control.xacro (robot description, xacro)
@@ -3,4 +3,5 @@
   <xacro:macro name="ur_ros2_control" params="name prefix
     use_fake_hardware:=false fake_sensor_commands:=false
+    initial_positions:=${dict(shoulder_pan_joint=0.0,shoulder_lift_joint=-1.57,elbow_joint=0.0,wrist_1_joint=-1.57,wrist_2_joint=0.0,wrist_3_joint=0.0)}
     script_filename output_recipe_filename
     input_recipe_filename tf_prefix
@@ -40,6 +41,6 @@
       <joint name="${prefix}shoulder_pan_joint">
         <command_interface name="position">
-          <param name="min">{-2*pi}</param>
-          <param name="max">{2*pi}</param>
+          <param name="min">${-2*pi}</param>
+          <param name="max">${2*pi}</param>
         </command_interface>
         <command_interface name="velocity">
@@ -50,10 +51,10 @@
         <state_interface name="velocity"/>
         <state_interface name="effort"/>
-        <param name="initial_position">0.0</param>  <!-- initial position for the FakeSystem -->
+        <param name="initial_position">${initial_positions['shoulder_pan_joint']}</param>  <!-- initial position for the FakeSystem -->
       </joint>
       <joint name="${prefix}shoulder_lift_joint">
         <command_interface name="position">
-          <param name="min">{-2*pi}</param>
-          <param name="max">{2*pi}</param>
+          <param name="min">${-2*pi}</param>
+          <param name="max">${2*pi}</param>
         </command_interface>
         <command_interface name="velocity">
@@ -64,10 +65,10 @@
         <state_interface name="velocity"/>
         <state_interface name="effort"/>
-        <param name="initial_position">-1.57</param>  <!-- initial position for the FakeSystem -->
+        <param name="initial_position">${initial_positions['shoulder_lift_joint']}</param>  <!-- initial position for the FakeSystem -->
       </joint>
       <joint name="${prefix}elbow_joint">
         <command_interface name="position">
-          <param name="min">{-pi}</param>
-          <param name="max">{pi}</param>
+          <param name="min">${-pi}</param>
+          <param name="max">${pi}</param>
         </command_interface>
         <command_interface name="velocity">
@@ -78,10 +79,10 @@
         <state_interface name="velocity"/>
         <state_interface name="effort"/>
-        <param name="initial_position">0.0</param>  <!-- initial position for the FakeSystem -->
+        <param name="initial_position">${initial_positions['elbow_joint']}</param>  <!-- initial position for the FakeSystem -->
       </joint>
       <joint name="${prefix}wrist_1_joint">
         <command_interface name="position">
-          <param name="min">{-2*pi}</param>
-          <param name="max">{2*pi}</param>
+          <param name="min">${-2*pi}</param>
+          <param name="max">${2*pi}</param>
         </command_interface>
         <command_interface name="velocity">
@@ -92,10 +93,10 @@
         <state_interface name="velocity"/>
         <state_interface name="effort"/>
-        <param name="initial_position">-1.57</param>  <!-- initial position for the FakeSystem -->
+        <param name="initial_position">${initial_positions['wrist_1_joint']}</param>  <!-- initial position for the FakeSystem -->
       </joint>
       <joint name="${prefix}wrist_2_joint">
         <command_interface name="position">
-          <param name="min">{-2*pi}</param>
-          <param name="max">{2*pi}</param>
+          <param name="min">${-2*pi}</param>
+          <param name="max">${2*pi}</param>
         </command_interface>
         <command_interface name="velocity">
@@ -106,10 +107,10 @@
         <state_interface name="velocity"/>
         <state_interface name="effort"/>
-        <param name="initial_position">0.0</param>  <!-- initial position for the FakeSystem -->
+        <param name="initial_position">${initial_positions['wrist_2_joint']}</param>  <!-- initial position for the FakeSystem -->
       </joint>
       <joint name="${prefix}wrist_3_joint">
         <command_interface name="position">
-          <param name="min">{-2*pi}</param>
-          <param name="max">{2*pi}</param>
+          <param name="min">${-2*pi}</param>
+          <param name="max">${2*pi}</param>
         </command_interface>
         <command_interface name="velocity">
@@ -120,5 +121,5 @@
         <state_interface name="velocity"/>
         <state_interface name="effort"/>
-        <param name="initial_position">0.0</param>  <!-- initial position for the FakeSystem -->
+        <param name="initial_position">${initial_positions['wrist_3_joint']}</param>  <!-- initial position for the FakeSystem -->
       </joint>
       <sensor name="tcp_fts_sensor">

File: ur_description/urdf/ur.urdf.xacro (robot description, xacro)
@@ -18,4 +18,7 @@
    <xacro:arg name="use_fake_hardware" default="false" />
    <xacro:arg name="fake_sensor_commands" default="false" />
+   <!-- initial position -->
+   <xacro:arg name="initial_positions_file" default="$(find ur_description)/config/initial_positions.yaml"/>
+   <xacro:property name="initial_positions_file" default="$(arg initial_positions_file)"/>
    <!-- arm -->
    <xacro:ur_robot
@@ -30,4 +33,5 @@
      safety_k_position="$(arg safety_k_position)"
      use_fake_hardware="$(arg use_fake_hardware)"
-     fake_sensor_commands="$(arg fake_sensor_commands)" />
+     fake_sensor_commands="$(arg fake_sensor_commands)"
+     initial_positions="${load_yaml(initial_positions_file)}" />
 </robot>

File: ur_description/urdf/ur_macro.xacro (robot description, xacro)
@@ -55,6 +55,6 @@
     safety_k_position:=20
     use_fake_hardware:=false
-    fake_sensor_commands:=false"
-  >
+    fake_sensor_commands:=false
+    initial_positions:=${dict(shoulder_pan_joint=0.0,shoulder_lift_joint=-1.57,elbow_joint=0.0,wrist_1_joint=-1.57,wrist_2_joint=0.0,wrist_3_joint=0.0)}">
     <!-- Load configuration data from the provided .yaml files -->
     <xacro:read_model_data
@@ -74,4 +74,5 @@
       name="URPositionHardwareInterface" prefix="${prefix}"
       use_fake_hardware="$(arg use_fake_hardware)"
+      initial_positions="${initial_positions}"
       fake_sensor_commands="$(arg fake_sensor_commands)"
       script_filename="$(arg script_filename)"
