Commit message: even more changes to add the bin picking kit

File: ur_description/urdf/ur_macro.xacro (robot description, xacro)
@@ -332,5 +332,5 @@
     <joint name="${prefix}flange-tool0" type="fixed">
       <!-- default toolframe - X+ left, Y+ up, Z+ front -->
-      <origin xyz="0 0 0" rpy="${pi/2.0} 0 ${pi/2.0}"/>
+      <origin xyz="0.3 0 0" rpy="${pi/2.0} 0 ${pi/2.0}"/>
       <parent link="${prefix}flange"/>
       <child link="${prefix}tool0"/>

Commit message: changes for adding gripper

File: ur_description/urdf/ur_macro.xacro (robot description, xacro)
@@ -332,5 +332,5 @@
     <joint name="${prefix}flange-tool0" type="fixed">
       <!-- default toolframe - X+ left, Y+ up, Z+ front -->
-      <origin xyz="0.3 0 0" rpy="${pi/2.0} 0 ${pi/2.0}"/>
+      <origin xyz="0.343 0 0" rpy="${pi/2.0} 0 ${pi/2.0}"/>
       <parent link="${prefix}flange"/>
       <child link="${prefix}tool0"/>

Commit message: copied config values from foxy_mowito

File: ur_description/urdf/ur_macro.xacro (robot description, xacro)
@@ -335,5 +335,5 @@
     <joint name="${prefix}flange-tool0" type="fixed">
       <!-- default toolframe - X+ left, Y+ up, Z+ front -->
-      <origin xyz="0 0 0" rpy="${pi/2.0} 0 ${pi/2.0}"/>
+      <origin xyz="0.343 0 0" rpy="${pi/2.0} 0 ${pi/2.0}"/>
       <parent link="${prefix}flange"/>
       <child link="${prefix}tool0"/>

Commit message: sv-- tool0 frame changed

File: ur_description/urdf/ur_macro.xacro (robot description, xacro)
@@ -332,6 +332,6 @@
     <link name="${prefix}tool0"/>
     <joint name="${prefix}flange-tool0" type="fixed">
-      <!-- default toolframe - X+ left, Y+ up, Z+ front -->
-      <origin xyz="0.343 0 0" rpy="${pi/2.0} 0 ${pi/2.0}"/>
+      <!-- default toolframe - X+ left, Y+ up, Z+ front --><!--sv - this convention does not hold anymore -->
+      <origin xyz="0.2949 0.0493 0" rpy="0 0 0"/>
       <parent link="${prefix}flange"/>
       <child link="${prefix}tool0"/>

Commit message: sv -- chcnaged config

File: ur_description/urdf/ur_macro.xacro (robot description, xacro)
@@ -333,8 +333,16 @@
     <joint name="${prefix}flange-tool0" type="fixed">
       <!-- default toolframe - X+ left, Y+ up, Z+ front --><!--sv - this convention does not hold anymore -->
-      <origin xyz="0.2949 0.0493 0" rpy="0 0 0"/>
+      <origin xyz="0.343 0 0" rpy="${pi/2.0} 0 ${pi/2.0}"/>
       <parent link="${prefix}flange"/>
       <child link="${prefix}tool0"/>
     </joint>
+    <!-- sv 'tool1' elbow joint -->
+    <link name="${prefix}tool1"/>
+    <joint name="${prefix}tool0-tool1" type="fixed">
+      <!-- default toolframe - X+ left, Y+ up, Z+ front --><!--sv - this convention does not hold anymore -->
+      <origin xyz="0.0493 0 -0.0481" rpy="0 0 0"/>
+      <parent link="${prefix}tool0"/>
+      <child link="${prefix}tool1"/>
+    </joint>
   </xacro:macro>
 </robot>

File: ur_moveit_config/srdf/ur_macro.srdf.xacro (robot description, xacro)
@@ -12,5 +12,5 @@
     <!--SUBGROUPS - Groups can also be formed by referencing to already defined group names-->
     <group name="${prefix}${name}_manipulator">
-      <chain base_link="${prefix}base_link" tip_link="${prefix}tool0" />
+      <chain base_link="${prefix}base_link" tip_link="${prefix}tool1" />
     </group>
     <!--GROUP STATES - Purpose - Define a named state for a particular group, in terms of joint values. This is useful to define states like 'folded arms'-->
@@ -48,4 +48,7 @@
     <disable_collisions link1="${prefix}tool0" link2="${prefix}wrist_2_link" reason="Never" />
     <disable_collisions link1="${prefix}tool0" link2="${prefix}wrist_3_link" reason="Adjacent" />
+    <disable_collisions link1="${prefix}tool1" link2="${prefix}wrist_1_link" reason="Never" />
+    <disable_collisions link1="${prefix}tool1" link2="${prefix}wrist_2_link" reason="Never" />
+    <disable_collisions link1="${prefix}tool1" link2="${prefix}wrist_3_link" reason="Adjacent" />
     <disable_collisions link1="${prefix}forearm_link" link2="${prefix}upper_arm_link" reason="Adjacent" />
     <disable_collisions link1="${prefix}forearm_link" link2="${prefix}wrist_1_link" reason="Adjacent" />

Commit message: sv -- need ti figure out exact tool tip, now working okish

File: ur_description/urdf/ur_macro.xacro (robot description, xacro)
@@ -341,5 +341,5 @@
     <joint name="${prefix}tool0-tool1" type="fixed">
       <!-- default toolframe - X+ left, Y+ up, Z+ front --><!--sv - this convention does not hold anymore -->
-      <origin xyz="0.0493 0 -0.0481" rpy="0 0 0"/>
+      <origin xyz="0.055 0.0233 -0.0526" rpy="0 0 0"/> <!--origin xyz="0.055,0.0233,-0.0526" rpy="0 0 0" -->
       <parent link="${prefix}tool0"/>
       <child link="${prefix}tool1"/>

Commit message: sv -- update config

File: ur_description/urdf/ur_macro.xacro (robot description, xacro)
@@ -341,5 +341,5 @@
     <joint name="${prefix}tool0-tool1" type="fixed">
       <!-- default toolframe - X+ left, Y+ up, Z+ front --><!--sv - this convention does not hold anymore -->
-      <origin xyz="0.055 0.0233 -0.0526" rpy="0 0 0"/> <!--origin xyz="0.055,0.0233,-0.0526" rpy="0 0 0" -->
+      <origin xyz="0.0492 0.0427 -0.0421" rpy="0 0 0"/> <!--origin xyz="0.055,0.0233,-0.0526" rpy="0 0 0" -->
       <parent link="${prefix}tool0"/>
       <child link="${prefix}tool1"/>

Commit message: sv -- new tooltip point, still not very accurate

File: ur_description/urdf/ur_macro.xacro (robot description, xacro)
@@ -341,5 +341,5 @@
     <joint name="${prefix}tool0-tool1" type="fixed">
       <!-- default toolframe - X+ left, Y+ up, Z+ front --><!--sv - this convention does not hold anymore -->
-      <origin xyz="0.0492 0.0427 -0.0421" rpy="0 0 0"/> <!--origin xyz="0.055,0.0233,-0.0526" rpy="0 0 0" -->
+      <origin xyz="0.0571 0.0353 -0.0305" rpy="0 0 0"/> <!--origin xyz="0.055,0.0233,-0.0526" rpy="0 0 0" -->
       <parent link="${prefix}tool0"/>
       <child link="${prefix}tool1"/>

Commit message: sv -- tooltip change

File: ur_description/urdf/ur_macro.xacro (robot description, xacro)
@@ -341,5 +341,5 @@
     <joint name="${prefix}tool0-tool1" type="fixed">
       <!-- default toolframe - X+ left, Y+ up, Z+ front --><!--sv - this convention does not hold anymore -->
-      <origin xyz="0.0571 0.0353 -0.0305" rpy="0 0 0"/> <!--origin xyz="0.055,0.0233,-0.0526" rpy="0 0 0" -->
+      <origin xyz="0.0547 0.0282 -0.0445" rpy="0 0 0"/> <!--origin xyz="0.055,0.0233,-0.0526" rpy="0 0 0" -->
       <parent link="${prefix}tool0"/>
       <child link="${prefix}tool1"/>

Commit message: sv -- added dummy tool1

File: ur_description/urdf/ur_macro.xacro (robot description, xacro)
@@ -337,4 +337,12 @@
       <child link="${prefix}tool0"/>
     </joint>
+    <!-- ROS-Industrial 'tool0' frame - all-zeros tool frame -->
+    <link name="${prefix}tool1"/>
+    <joint name="${prefix}tool0-tool1" type="fixed">
+      <!-- default toolframe - X+ left, Y+ up, Z+ front -->
+      <origin xyz="0.0 0 0" rpy="0.0 0 0.0"/>
+      <parent link="${prefix}tool0"/>
+      <child link="${prefix}tool1"/>
+    </joint>
   </xacro:macro>
 </robot>

File: ur_moveit_config/srdf/ur_macro.srdf.xacro (robot description, xacro)
@@ -12,5 +12,5 @@
     <!--SUBGROUPS - Groups can also be formed by referencing to already defined group names-->
     <group name="${prefix}${name}_manipulator">
-      <chain base_link="${prefix}base_link" tip_link="${prefix}tool0" />
+      <chain base_link="${prefix}base_link" tip_link="${prefix}tool1" />
     </group>
     <!--GROUP STATES - Purpose - Define a named state for a particular group, in terms of joint values. This is useful to define states like 'folded arms'-->

Commit message: sv -- demo

File: ur_description/urdf/ur_macro.xacro (robot description, xacro)
@@ -333,5 +333,5 @@
     <joint name="${prefix}flange-tool0" type="fixed">
       <!-- default toolframe - X+ left, Y+ up, Z+ front -->
-      <origin xyz="0.343 0 0" rpy="${pi/2.0} 0 ${pi/2.0}"/>
+      <origin xyz="0.423 0 0" rpy="${pi/2.0} 0 ${pi/2.0}"/>
       <parent link="${prefix}flange"/>
       <child link="${prefix}tool0"/>

Commit message: kb chencing out

File: ur_description/urdf/ur_macro.xacro (robot description, xacro)
@@ -333,5 +333,5 @@
     <joint name="${prefix}flange-tool0" type="fixed">
       <!-- default toolframe - X+ left, Y+ up, Z+ front -->
-      <origin xyz="0.423 0 0" rpy="${pi/2.0} 0 ${pi/2.0}"/>
+      <origin xyz="0.483 0 0" rpy="${pi/2.0} 0 ${pi/2.0}"/>
       <parent link="${prefix}flange"/>
       <child link="${prefix}tool0"/>

Commit message: sv - longer pipe

File: ur_description/urdf/ur_macro.xacro (robot description, xacro)
@@ -333,5 +333,5 @@
     <joint name="${prefix}flange-tool0" type="fixed">
       <!-- default toolframe - X+ left, Y+ up, Z+ front -->
-      <origin xyz="0.483 0 0" rpy="${pi/2.0} 0 ${pi/2.0}"/>
+      <origin xyz="0.400 0 0" rpy="${pi/2.0} 0 ${pi/2.0}"/>
       <parent link="${prefix}flange"/>
       <child link="${prefix}tool0"/>

Commit message: kb added transformation from flange to camera_optical_color_frame in ur5e urdf macro

File: ur_description/urdf/ur_macro.xacro (robot description, xacro)
@@ -333,7 +333,14 @@
     <joint name="${prefix}flange-tool0" type="fixed">
       <!-- default toolframe - X+ left, Y+ up, Z+ front -->
-      <origin xyz="0.400 0 0" rpy="${pi/2.0} 0 ${pi/2.0}"/>
+      <origin xyz="0.600 0 0" rpy="${pi/2.0} 0 ${pi/2.0}"/>
       <parent link="${prefix}flange"/>
       <child link="${prefix}tool0"/>
+    </joint>
+    <link name="${prefix}camera_color_optical_frame"/>
+    <joint name="${prefix}flange-camera_color_optical_frame" type="fixed">
+      <!-- default toolframe - X+ left, Y+ up, Z+ front -->
+      <origin xyz="0.0358305850983095 0.024214241762794915 -0.08249533085075297" rpy="-2.4057309 1.5051829 -1.5154178"/>
+      <parent link="${prefix}flange"/>
+      <child link="${prefix}camera_color_optical_frame"/>
     </joint>
     <!-- ROS-Industrial 'tool0' frame - all-zeros tool frame -->

Commit message: kb chnages to urdf for camera to wrist 3 link transform

File: ur_description/urdf/ur_macro.xacro (robot description, xacro)
@@ -337,9 +337,14 @@
       <child link="${prefix}tool0"/>
     </joint>
+    <link name="${prefix}camera_color_optical_frame1"/>
+    <joint name="${prefix}wrist_3-camera_color_optical_frame1" type="fixed">
+      <origin xyz="0.025 -0.082 0.034" rpy="0.0035171 0.0642818 0.7902383"/>
+      <parent link="${prefix}wrist_3_link"/>
+      <child link="${prefix}camera_color_optical_frame1"/>
+    </joint>
     <link name="${prefix}camera_color_optical_frame"/>
-    <joint name="${prefix}flange-camera_color_optical_frame" type="fixed">
-      <!-- default toolframe - X+ left, Y+ up, Z+ front -->
-      <origin xyz="0.0358305850983095 0.024214241762794915 -0.08249533085075297" rpy="-2.4057309 1.5051829 -1.5154178"/>
-      <parent link="${prefix}flange"/>
+    <joint name="${prefix}tool0-camera_color_optical_frame" type="fixed">
+      <origin xyz="0.025316732076068958 -0.08219936857804473 -0.5655037992448424" rpy="0.0475148 0.0432808 0.7909686"/>
+      <parent link="${prefix}tool0"/>
       <child link="${prefix}camera_color_optical_frame"/>
     </joint>

Commit message: kb all chages done

File: ur_description/urdf/ur_macro.xacro (robot description, xacro)
@@ -331,21 +331,27 @@
     <!-- ROS-Industrial 'tool0' frame - all-zeros tool frame -->
     <link name="${prefix}tool0"/>
-    <joint name="${prefix}flange-tool0" type="fixed">
+    <joint name="${prefix}wrist_3-tool0" type="fixed">
       <!-- default toolframe - X+ left, Y+ up, Z+ front -->
-      <origin xyz="0.600 0 0" rpy="${pi/2.0} 0 ${pi/2.0}"/>
-      <parent link="${prefix}flange"/>
+      <origin xyz="-0.023 0.016 0.318" rpy="-0.0511685 0.0285234 2.3987783"/>
+      <parent link="${prefix}wrist_3_link"/>
       <child link="${prefix}tool0"/>
     </joint>
     <link name="${prefix}camera_color_optical_frame1"/>
     <joint name="${prefix}wrist_3-camera_color_optical_frame1" type="fixed">
-      <origin xyz="0.025 -0.082 0.034" rpy="0.0035171 0.0642818 0.7902383"/>
+      <origin xyz="0.023951330579827648 -0.08148942116607773 0.03379282985859283" rpy="0.0478417 0.0445253 0.7901463"/>
       <parent link="${prefix}wrist_3_link"/>
       <child link="${prefix}camera_color_optical_frame1"/>
     </joint>
-    <link name="${prefix}camera_color_optical_frame"/>
-    <joint name="${prefix}tool0-camera_color_optical_frame" type="fixed">
-      <origin xyz="0.025316732076068958 -0.08219936857804473 -0.5655037992448424" rpy="0.0475148 0.0432808 0.7909686"/>
+    <link name="${prefix}realsense_frame"/>
+    <joint name="${prefix}camera_color_optical_frame1-realsense_frame" type="fixed">
+      <origin xyz="0 0 0" rpy="0 0 0"/>
+      <parent link="${prefix}camera_color_optical_frame1"/>
+      <child link="${prefix}realsense_frame"/>
+    </joint>
+    <link name="${prefix}camera_color_optical_frame11"/>
+    <joint name="${prefix}tool0-camera_color_optical_frame11" type="fixed">
+      <origin xyz="-0.097 0.024 -0.287" rpy="-0.0132149 -0.064089 -1.6079909"/>
       <parent link="${prefix}tool0"/>
-      <child link="${prefix}camera_color_optical_frame"/>
+      <child link="${prefix}camera_color_optical_frame11"/>
     </joint>
     <!-- ROS-Industrial 'tool0' frame - all-zeros tool frame -->

Commit message: sv -- calib testing

File: ur_description/urdf/ur_macro.xacro (robot description, xacro)
@@ -333,5 +333,5 @@
     <joint name="${prefix}wrist_3-tool0" type="fixed">
       <!-- default toolframe - X+ left, Y+ up, Z+ front -->
-      <origin xyz="-0.023 0.016 0.318" rpy="-0.0511685 0.0285234 2.3987783"/>
+      <origin xyz="0 0 0.318" rpy="-0.0511685 0.0285234 2.3987783"/>
       <parent link="${prefix}wrist_3_link"/>
       <child link="${prefix}tool0"/>

Commit message: sv -- removed compliance gripper

File: ur_description/urdf/ur_macro.xacro (robot description, xacro)
@@ -341,5 +341,5 @@
     <joint name="${prefix}tool0-tool1" type="fixed">
       <!-- default toolframe - X+ left, Y+ up, Z+ front -->
-      <origin xyz="0.0 0 0" rpy="0.0 0 0.0"/>
+      <origin xyz="0.0 0 0.0" rpy="0.0 0 0.0"/>
       <parent link="${prefix}tool0"/>
       <child link="${prefix}tool1"/>
